Commit message: debug drone sim expert add line world generator clean up test fsm clean up robot mapper add condor launcher for line world

File: src/sim/ros/gazebo/urdf/drone_sim.gazebo.xacro (robot description, xacro)
@@ -1,7 +1,6 @@
 <?xml version="1.0"?>
 <robot name="quadrotor" xmlns:xacro="http://www.ros.org/wiki/xacro">
-		<xacro:include filename="$(find hector_quadrotor_description)/urdf/quadrotor_with_kinect_and_lidar.urdf.xacro" />
-    <!-- <xacro:include filename="$(find hector_quadrotor_description)/urdf/quadrotor_with_cam_and_kinect.urdf.xacro" /> -->
-    <!-- <xacro:include filename="$(find hector_quadrotor_description)/urdf/quadrotor.urdf.xacro" /> -->
-    <xacro:include filename="$(find hector_quadrotor_gazebo)/urdf/quadrotor_plugins.gazebo.xacro" />
+<!--		<xacro:include filename="$(find hector_quadrotor_description)/urdf/quadrotor_with_kinect_and_lidar.urdf.xacro" />-->
+		<xacro:include filename="$(env HOME)/src/sim/ros/gazebo/urdf/drone_sim.urdf.xacro" />
+        <xacro:include filename="$(find hector_quadrotor_gazebo)/urdf/quadrotor_plugins.gazebo.xacro" />
 </robot>

File: src/sim/ros/gazebo/urdf/drone_sim.urdf.xacro (robot description, xacro)
@@ -1,9 +1,32 @@
 <?xml version="1.0"?>
 <robot
-  name="quadrotor"
-  xmlns:xacro="http://www.ros.org/wiki/xacro"
+    name="quadrotor"
+    xmlns:xacro="http://www.ros.org/wiki/xacro"
 >
+     <xacro:property name="M_PI" value="3.1415926535897931" />
     <!-- Included URDF Files -->
-    <xacro:include filename="$(find hector_quadrotor_description)/urdf/quadrotor_base.urdf.xacro" />
+    <xacro:include filename="bebop.urdf.xacro" />
+    <!-- Forward facing camera-->
+    <xacro:include filename="$(find hector_sensors_description)/urdf/generic_camera.urdf.xacro" />
+    <xacro:generic_camera name="down_cam"
+                          parent="base_link"
+                          ros_topic="camera/image"
+                          cam_info_topic="camera/camera_info"
+                          update_rate="10"
+                          res_x="128"
+                          res_y="128"
+                          image_format="R8G8B8" hfov="80">
+      <origin xyz="0.05 0.0 -0.1" rpy="0 ${80*pi/180} 0"/>
+    </xacro:generic_camera>
+    <!-- Kinect Camera -->
+<!--    <include filename="$(find hector_quadrotor_description)/urdf/kinect_camera.urdf.xacro" />-->
+<!--    <xacro:kinect_camera name="kinect" parent="base_link">-->
+<!--      <origin xyz="0.1 0.0 0.1" rpy="0 0 0"/>-->
+<!--    </xacro:kinect_camera>-->
+    <!-- Lidar Camera -->
+<!--    <include filename="$(find hector_quadrotor_description)/urdf/lidar.urdf.xacro" />-->
+<!--    <xacro:lidar name="lidar" parent="base_link">-->
+<!--      <origin xyz="0.1 0.0 0.5" rpy="0 0 0"/>-->
+<!--    </xacro:lidar>-->
     <!-- Instantiate quadrotor_base_macro once (has no parameters atm) -->
     <xacro:quadrotor_base_macro />

File: src/sim/ros/gazebo/urdf/wide_angle_camera.urdf.xacro (robot description, xacro)
@@ -44,7 +44,6 @@
           <update_rate>10.0</update_rate>
           <camera name="head">
-            <!-- 106 degrees horizontal field of view -->
+            <!-- degrees horizontal field of view -->
             <horizontal_fov>3.14</horizontal_fov>
-<!--            <horizontal_fov>6</horizontal_fov>-->
             <vertical_fov>3.14</vertical_fov>
             <image>
