Commit message: create double sim drone robot config, test in launch, switch in robot according to name instead of if statements, add seperate down cam and wide angle drone model

File: src/sim/ros/gazebo/urdf/drone_sim_down_cam.gazebo.xacro (robot description, xacro)
@@ -1,5 +1,5 @@
 <?xml version="1.0"?>
 <robot name="quadrotor" xmlns:xacro="http://www.ros.org/wiki/xacro">
-		<xacro:include filename="$(env CODEDIR)/src/sim/ros/gazebo/urdf/drone_sim.urdf.xacro" />
+		<xacro:include filename="$(env CODEDIR)/src/sim/ros/gazebo/urdf/drone_sim_down_cam.urdf.xacro" />
         <xacro:include filename="$(find hector_quadrotor_gazebo)/urdf/quadrotor_plugins.gazebo.xacro" />
 </robot>

File: src/sim/ros/gazebo/urdf/drone_sim_down_cam.urdf.xacro (robot description, xacro)
@@ -9,13 +9,13 @@
     <!-- Forward facing camera-->
     <xacro:include filename="$(find hector_sensors_description)/urdf/generic_camera.urdf.xacro" />
-    <xacro:generic_camera name="forward"
+    <xacro:generic_camera name="down"
                           parent="base_link"
                           ros_topic="camera/image"
                           cam_info_topic="camera/camera_info"
                           update_rate="10"
-                          res_x="200"
-                          res_y="200"
+                          res_x="128"
+                          res_y="128"
                           image_format="R8G8B8" hfov="80">
-      <origin xyz="0.05 0.0 -0.1" rpy="0 0 0"/>
+      <origin xyz="0.05 0.0 -0.1" rpy="0 ${90*pi/180} 0"/>
     </xacro:generic_camera>
     <!-- Kinect Camera -->
@@ -25,8 +25,8 @@
 <!--    </xacro:kinect_camera>-->
     <!-- Lidar Camera -->
-    <include filename="$(find hector_quadrotor_description)/urdf/lidar.urdf.xacro" />
-    <xacro:lidar name="lidar" parent="base_link">
-      <origin xyz="0.1 0.0 0.5" rpy="0 0 0"/>
-    </xacro:lidar>
+<!--    <include filename="$(find hector_quadrotor_description)/urdf/lidar.urdf.xacro" />-->
+<!--    <xacro:lidar name="lidar" parent="base_link">-->
+<!--      <origin xyz="0.1 0.0 0.5" rpy="0 0 0"/>-->
+<!--    </xacro:lidar>-->
     <!-- Instantiate quadrotor_base_macro once (has no parameters atm) -->
     <xacro:quadrotor_base_macro />

File: src/sim/ros/gazebo/urdf/drone_sim_wide_angle.gazebo.xacro (robot description, xacro)
@@ -1,5 +1,5 @@
 <?xml version="1.0"?>
 <robot name="quadrotor" xmlns:xacro="http://www.ros.org/wiki/xacro">
-		<xacro:include filename="$(env CODEDIR)/src/sim/ros/gazebo/urdf/drone_sim.urdf.xacro" />
+		<xacro:include filename="$(env CODEDIR)/src/sim/ros/gazebo/urdf/drone_sim_wide_angle.urdf.xacro" />
         <xacro:include filename="$(find hector_quadrotor_gazebo)/urdf/quadrotor_plugins.gazebo.xacro" />
 </robot>

File: src/sim/ros/gazebo/urdf/drone_sim_wide_angle.urdf.xacro (robot description, xacro)
@@ -16,5 +16,5 @@
                           res_x="200"
                           res_y="200"
-                          image_format="R8G8B8" hfov="80">
+                          image_format="R8G8B8" hfov="120">
       <origin xyz="0.05 0.0 -0.1" rpy="0 0 0"/>
     </xacro:generic_camera>
@@ -25,8 +25,8 @@
 <!--    </xacro:kinect_camera>-->
     <!-- Lidar Camera -->
-    <include filename="$(find hector_quadrotor_description)/urdf/lidar.urdf.xacro" />
-    <xacro:lidar name="lidar" parent="base_link">
-      <origin xyz="0.1 0.0 0.5" rpy="0 0 0"/>
-    </xacro:lidar>
+<!--    <include filename="$(find hector_quadrotor_description)/urdf/lidar.urdf.xacro" />-->
+<!--    <xacro:lidar name="lidar" parent="base_link">-->
+<!--      <origin xyz="0.1 0.0 0.5" rpy="0 0 0"/>-->
+<!--    </xacro:lidar>-->
     <!-- Instantiate quadrotor_base_macro once (has no parameters atm) -->
     <xacro:quadrotor_base_macro />
