Commit message: drone sim 90 degrees down

File: src/sim/ros/gazebo/urdf/drone_sim.urdf.xacro (robot description, xacro)
@@ -17,5 +17,5 @@
                           res_y="128"
                           image_format="R8G8B8" hfov="80">
-      <origin xyz="0.05 0.0 -0.1" rpy="0 ${80*pi/180} 0"/>
+      <origin xyz="0.05 0.0 -0.1" rpy="0 ${90*pi/180} 0"/>
     </xacro:generic_camera>
     <!-- Kinect Camera -->

Commit message: adjust double drone camera and control mapper to handle arbitrary configs and commands

File: src/sim/ros/gazebo/urdf/drone_sim.urdf.xacro (robot description, xacro)
@@ -27,5 +27,5 @@
     <include filename="$(find hector_quadrotor_description)/urdf/lidar.urdf.xacro" />
     <xacro:lidar name="lidar" parent="base_link">
-      <origin xyz="0.1 0.0 0.5" rpy="0 0 0"/>
+      <origin xyz="0.1 0.0 0.1" rpy="0 0 0"/>
     </xacro:lidar>
     <!-- Instantiate quadrotor_base_macro once (has no parameters atm) -->

File: src/sim/ros/gazebo/urdf/drone_sim_wide_angle.urdf.xacro (robot description, xacro)
@@ -17,5 +17,5 @@
                           res_y="200"
                           image_format="R8G8B8" hfov="120">
-      <origin xyz="0.05 0.0 -0.1" rpy="0 0 0"/>
+      <origin xyz="0.1 0.0 0.1" rpy="0 0 0"/>
     </xacro:generic_camera>
     <!-- Kinect Camera -->

Commit message: add chessboard world and model, adjust camera tilt to mimic bebop, add test chessboard

File: src/sim/ros/gazebo/urdf/drone_sim.urdf.xacro (robot description, xacro)
@@ -14,8 +14,8 @@
                           cam_info_topic="camera/camera_info"
                           update_rate="10"
-                          res_x="200"
-                          res_y="200"
+                          res_x="856"
+                          res_y="480"
                           image_format="R8G8B8" hfov="80">
-      <origin xyz="0.05 0.0 -0.1" rpy="0 0 0"/>
+      <origin xyz="0.05 0.0 -0.1" rpy="0 0.2267 0"/>
     </xacro:generic_camera>
     <!-- Kinect Camera -->

Commit message: add april tags reset mathias controller

File: src/sim/ros/gazebo/urdf/drone_sim.urdf.xacro (robot description, xacro)
@@ -25,8 +25,8 @@
 <!--    </xacro:kinect_camera>-->
     <!-- Lidar Camera -->
-    <include filename="$(find hector_quadrotor_description)/urdf/lidar.urdf.xacro" />
-    <xacro:lidar name="lidar" parent="base_link">
-      <origin xyz="0.1 0.0 0.1" rpy="0 0 0"/>
-    </xacro:lidar>
+<!--    <include filename="$(find hector_quadrotor_description)/urdf/lidar.urdf.xacro" />-->
+<!--    <xacro:lidar name="lidar" parent="base_link">-->
+<!--      <origin xyz="0.1 0.0 0.1" rpy="0 0 0"/>-->
+<!--    </xacro:lidar>-->
     <!-- Instantiate quadrotor_base_macro once (has no parameters atm) -->
     <xacro:quadrotor_base_macro />
