Commit message: adjust inertia params, higher turn threshold, more tests

File: src/sim/ros/gazebo/urdf/bebop.urdf.xacro (robot description, xacro)
@@ -9,5 +9,5 @@
         <mass value="0.5" />
         <origin xyz="0 0 0.1" />
-        <inertia ixx="0.01152" ixy="0.0" ixz="0.0" iyy="0.01152" iyz="0.0" izz="0.0218" />
+        <inertia ixx="0.00389" ixy="0.0" ixz="0.0" iyy="0.00389" iyz="0.0" izz="0.0078" />
       </inertial>
       <visual>

Commit message: add extra inertia option (no visible difference)

File: src/sim/ros/gazebo/urdf/bebop.urdf.xacro (robot description, xacro)
@@ -9,5 +9,6 @@
         <mass value="0.5" />
         <origin xyz="0 0 0.1" />
-        <inertia ixx="0.00389" ixy="0.0" ixz="0.0" iyy="0.00389" iyz="0.0" izz="0.0078" />
+<!--        <inertia ixx="0.00389" ixy="0.0" ixz="0.0" iyy="0.00389" iyz="0.0" izz="0.0078" />-->
+        <inertia ixx="0.01152" ixy="0.0" ixz="0.0" iyy="0.01152" iyz="0.0" izz="0.0218" />
       </inertial>
       <visual>

Commit message: Add bebop mesh

File: src/sim/ros/gazebo/urdf/bebop.urdf.xacro (robot description, xacro)
@@ -13,8 +13,9 @@
       </inertial>
       <visual>
-        <origin xyz="0 0 0" rpy="0 0 3.14" />
+        <origin xyz="0 0 0" rpy="0 0 0" />
         <geometry>
           <!-- <mesh filename="package://hector_quadrotor_description/meshes/ardrone/quadrotor_4.dae"/> -->
-          <mesh filename="package://hector_quadrotor_description/meshes/bebop/quadrotor_CAD.dae"/>
+<!--          <mesh filename="package://hector_quadrotor_description/meshes/bebop/quadrotor_CAD.dae"/>-->
+          <mesh filename="../models/parrot_bebop_2/meshes/hull.dae"/>
         </geometry>
       </visual>

Commit message: setup data_generation script for gate_cone_line

File: src/sim/ros/gazebo/urdf/bebop.urdf.xacro (robot description, xacro)
@@ -17,5 +17,5 @@
           <!-- <mesh filename="package://hector_quadrotor_description/meshes/ardrone/quadrotor_4.dae"/> -->
 <!--          <mesh filename="package://hector_quadrotor_description/meshes/bebop/quadrotor_CAD.dae"/>-->
-          <mesh filename="../models/parrot_bebop_2/meshes/hull.dae"/>
+          <mesh filename="$(env CODEDIR)/src/sim/ros/gazebo/models/parrot_bebop_2/meshes/hull.dae"/>
         </geometry>
       </visual>
